File: corne-ultralight/pcb/corne-ultralight.kicad_sch (KiCad schematic)
At the start: 102 parts, among them J2 OLED, J7 OLED, SW1 SW_PUSH, SW10 SW_PUSH, SW11 SW_PUSH, SW12 SW_PUSH, SW13 SW_PUSH, SW14 SW_PUSH, SW15 SW_PUSH, SW16 SW_PUSH, SW17 SW_PUSH, SW18 SW_PUSH, SW19 SW_PUSH, SW2 SW_PUSH, SW20 SW_PUSH, SW21 SW_PUSH, SW22 SW_PUSH, SW23 SW_PUSH, SW24 SW_PUSH, SW25 SW_PUSH, SW26 SW_PUSH, SW27 SW_PUSH, SW28 SW_PUSH, SW29 SW_PUSH, SW3 SW_PUSH, SW30 SW_PUSH, SW31 SW_PUSH, SW32 SW_PUSH, SW33 SW_PUSH, SW34 SW_PUSH, SW35 SW_PUSH, SW36 SW_PUSH, SW37 SW_PUSH, SW38 SW_PUSH, SW39 SW_PUSH, SW4 SW_PUSH, SW40 SW_PUSH, SW41 SW_PUSH, SW42 SW_PUSH, SW5 SW_PUSH, SW6 SW_PUSH, SW7 SW_PUSH, SW8 SW_PUSH, SW9 SW_PUSH, U1 ProMicro, U2 ProMicro

Commit message: added hotswap
Parts:
- SW9: footprint gateron-ks27:gateron-ks27-choc-v1 -> kbd:CherryMX_ChocV2_1u
Changed lines of the file:
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@@
     (property "Reference" "SW9" (id 0) (at 62.865 36.576 0))
     (property "Value" "SW_PUSH" (id 1) (at 59.055 41.402 0))
-    (property "Footprint" "gateron-ks27:gateron-ks27-choc-v1" (id 2) (at 59.055 39.37 0)
+    (property "Footprint" "kbd:CherryMX_ChocV2_1u" (id 2) (at 59.055 39.37 0)
       (effects (font (size 1.27 1.27)) hide)
     )
@@
     )
     (path "/00000000-0000-0000-0000-00005a5e2d32"
-      (reference "SW9") (unit 1) (value "SW_PUSH") (footprint "gateron-ks27:gateron-ks27-choc-v1")
+      (reference "SW9") (unit 1) (value "SW_PUSH") (footprint "kbd:CherryMX_ChocV2_1u")
     )
     (path "/00000000-0000-0000-0000-00005a5e2d3e"
